File: ESP32_project.kicad_sch (KiCad schematic)
At the start: 24 parts, among them SW1 KMR2, SW2 KMR2, U1 AP2112-3.3, X1 ESP32_WROOM32, X2 JSTPH

Commit message: Remove diodes and switch
Parts:
- removed D1, D2: 1n4148, Adafruit ESP32 Huzzah Breakout:SOD-323, symbol Adafruit ESP32 Huzzah Breakout-eagle-import:DIODESOD-323
- removed SW2: KMR2, Adafruit ESP32 Huzzah Breakout:BTN_KMR2_4.6X2.8, symbol Adafruit ESP32 Huzzah Breakout-eagle-import:SWITCH_TACT_SMT4.6X2.8
